File: signal_generator_evb_v2/signal_generator_evb.kicad_pcb (KiCad board)
At the start: 4 copper layers, 28 x 65 mm, 69 parts, among them J2 Conn_Coaxial, J3 Conn_Coaxial, J4 Conn_Coaxial, J5 Conn_Coaxial, J6 Conn_01x04_Pin, SW1 RotaryEncoder_Switch_MP, SW2 SW_Push, SW3 SW_Push, SW4 SW_Push, U2 CH32V003FxUx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

Commit message: 250801_0030
Parts:
- moved C16 2.16 mm to (97.0, 78.0), turned to 45 degrees
- moved R13 1.47 mm to (103.8, 70.2), turned to 135 degrees
- moved C19 1.31 mm to (100.5, 72.2), turned to -45 degrees
- moved C15 1.17 mm to (100.3, 78.2), turned to 135 degrees
- moved Y1 0.62 mm to (98.7, 79.1), turned to 135 degrees
- moved C20 0.57 mm to (103.8, 72.3), turned to -135 degrees
- moved Y3 0.18 mm to (102.1, 71.2), turned to 135 degrees
Routing:
- net Net-(C20-Pad1): track 5.61 -> 2.81 mm
- net Net-(Y2-XB): track 4.16 -> 6.82 mm
- net GND: track 45.4 -> 43.8 mm, vias 50 -> 59
- net +3V3: track 117.4 -> 116.1 mm
- net Net-(Y2-XA): track 6.81 -> 5.63 mm
- net Net-(U2-PA1): track 4.23 -> 5.05 mm
- net Net-(U2-PA2): track 1.44 -> 2.21 mm
- added copper zone on B.Cu, net +5V
- added copper zone on In1.Cu, net +5V
